Commit message: CV5

File: install/rrm_simple_robot_model/share/rrm_simple_robot_model/urdf/arm.urdf (robot description, URDF)
Before this commit: robot arm, 6 links, 5 joints
Links:
- added link link_3_4; visual sphere radius=0.02
- added link link_4; visual cylinder length=0.05 radius=0.01
- added link link_4_5; visual sphere radius=0.02
- added link link_5; visual cylinder length=0.15 radius=0.01
- added link link_5_6; visual sphere radius=0.02
- added link link_6; visual cylinder length=0.1 radius=0.012
- link link_2: geometry visual cylinder length=0.203 radius=0.01
- link link_2_3: geometry visual sphere radius=0.02
Joints:
- removed joint joint_3-tool0
- added joint joint_3_4_fixed: type fixed, parent link_3, child link_3_4, origin xyz=0 0 0.203 rpy=0 0 0
- added joint joint_4: type revolute, parent link_3, child link_4, origin xyz=0 0 0.203 rpy=0 0 0, axis 0 0 1, limit lower=-3.14 upper=3.14 effort=1000.0 velocity=0.5
- added joint joint_4_5_fixed: type fixed, parent link_4, child link_4_5, origin xyz=0 0 0.05 rpy=0 0 0
- added joint joint_5: type revolute, parent link_4, child link_5, origin xyz=0 0 0.05 rpy=0 0 0, axis 0 1 0, limit lower=-2.2 upper=2.2 effort=1000.0 velocity=0.5
- added joint joint_5_6_fixed: type fixed, parent link_5, child link_5_6, origin xyz=0 0 0.15 rpy=0 0 0
- added joint joint_6: type prismatic, parent link_5, child link_6, origin xyz=0 0 0.15 rpy=0 0 0, axis 0 0 1, limit lower=0 upper=0.1 effort=1000.0 velocity=0.5
- added joint joint_6_tool0: type fixed, parent link_6, child tool0, origin xyz=0 0 0.1 rpy=0 0 0
