Commit message: CV6 - Back to 3DOF

File: src/cv2/rrm_simple_robot_model/urdf/arm.urdf (robot description, URDF)
Before this commit: robot arm, 12 links, 11 joints
Links:
- removed link link_3_4
- removed link link_4
- removed link link_4_5
- removed link link_5
- removed link link_5_6
- removed link link_6
- link link_2: geometry visual cylinder length=0.178 radius=0.01
- link link_2_3: geometry visual sphere radius=0.03
Joints:
- removed joint joint_3_4_fixed
- removed joint joint_4
- removed joint joint_4_5_fixed
- removed joint joint_5
- removed joint joint_5_6_fixed
- removed joint joint_6
- removed joint joint_6_tool0
- added joint joint_3-tool0: type fixed, parent link_3, child tool0, origin xyz=0 0 0.203 rpy=0 0 0
